Commit message: feb 11

File: robots/rb5_850e.urdf (robot description, URDF)
Before this commit: robot rb5_850e, 9 links, 8 joints
Joints:
- joint tcp_joint: origin xyz=0 -0.0967 0 rpy=0 0 0 -> xyz=0 -0.1 0.1 rpy=0 0 0

Commit message: have problem that value is nan

File: robots/rb5_850e.urdf (robot description, URDF)
Before this commit: robot rb5_850e, 9 links, 8 joints
Joints:
- joint tcp_joint: origin xyz=0 -0.1 0.1 rpy=0 0 0 -> xyz=0 -0.11 0.1 rpy=0 0 0
